Commit message: final merge

File: urdf/yz_41dof.urdf (robot description, URDF)
Before this commit: robot snakebot, 76 links, 75 joints
Joints:
- joint attach-base: origin (none) -> xyz=0 0 0 rpy=0 0 0
- joint attach-flange: origin (none) -> xyz=0 0 0 rpy=0 0 0
- joint attach-mating-plate: origin (none) -> xyz=0 0 0 rpy=0 0 0

File: urdf/yz_9dof.urdf (robot description, URDF)
Before this commit: robot snakebot, 28 links, 27 joints
Joints:
- joint attach-base: origin (none) -> xyz=0 0 0 rpy=0 0 0
- joint attach-flange: origin (none) -> xyz=0 0 0 rpy=0 0 0
- joint attach-mating-plate: origin (none) -> xyz=0 0 0 rpy=0 0 0
